Commit message: adding lidar sensor

File: workspace/src/dirac_description/urdf/dirac.urdf (robot description, URDF)
Before this commit: robot dirac, 6 links, 5 joints
Links:
- added link lidar_link, mass 0.5; collision cylinder length=0.1 radius=0.05; visual cylinder length=0.1 radius=0.05
Joints:
- added joint lidar_joint: type fixed, parent link_chassis, child lidar_link, origin xyz=0 0 0.25 rpy=0 0 0

Commit message: scale robot size down

File: workspace/src/dirac_description/urdf/dirac.urdf (robot description, URDF)
Before this commit: robot dirac, 7 links, 6 joints
Links:
- link link_chassis: geometry collision box size=0.35 0.35 0.14; visual box size=0.35 0.35 0.14
Joints:
- joint left_wheel_hinge_back: origin xyz=-0.2 0.30 0 rpy=0 0 0 -> xyz=-0.14 0.21 0 rpy=0 0 0
- joint left_wheel_hinge_front: origin xyz=0.2 0.30 0 rpy=0 0 0 -> xyz=0.14 0.21 0 rpy=0 0 0
- joint lidar_joint: origin xyz=0 0 0.25 rpy=0 0 0 -> xyz=0 0 0.175 rpy=0 0 0
- joint right_wheel_hinge_back: origin xyz=-0.2 -0.30 0 rpy=0 0 0 -> xyz=-0.14 -0.21 0 rpy=0 0 0
- joint right_wheel_hinge_front: origin xyz=0.2 -0.30 0 rpy=0 0 0 -> xyz=0.14 -0.21 0 rpy=0 0 0
